Commit message: Fake sourccey arm teleop semi predictably responsive

File: lerobot/common/robots/sourccey_v2beta/model/Arm.urdf (robot description, URDF)
Before this commit: robot Arm, 17 links, 14 joints
Joints:
- removed joint Arm-Base-V3-v1_Rigid-1
- removed joint Arm-Bicep-v1_Rigid-6
- removed joint Arm-Forearm-v1_Rigid-8
- removed joint Arm-Wrist-v1_Rigid-10
- removed joint Feetech-Servo-Motor-v1-1_Revolute-5
- removed joint Feetech-Servo-Motor-v1-2_Revolute-7
- removed joint Feetech-Servo-Motor-v1-3_Revolute-9
- removed joint Feetech-Servo-Motor-v1-4_Revolute-11
- removed joint Feetech-Servo-Motor-v1_Revolute-2
- removed joint Gripper-Base-Back-v1_Rigid-12
- removed joint Gripper-Base-Back-v1_Rigid-13
- removed joint Gripper-Base-Front-Angled-Camera-v1_Slider-14
- removed joint Gripper-Base-Front-Angled-Camera-v1_Slider-15
- removed joint Shoulder-With-Gearbox-V3-v1_Rigid-4

Commit message: Adding the semi working so100 urdf

File: lerobot/common/robots/sourccey_v2beta/model/Arm.urdf (robot description, URDF)
Before this commit: robot Arm, 17 links, 0 joints
Joints:
- added joint Arm-Base-V3-v1_Rigid-1: type fixed, parent Arm-Base-V3-v1, child Feetech-Servo-Motor-v1, origin xyz=0.05233622014901163 6.859801863787153e-19 -0.024715040894069628 rpy=-8.031609262326351e-32 -1.5707963267948828 0
- added joint Arm-Bicep-v1_Rigid-6: type fixed, parent Arm-Bicep-v1, child Feetech-Servo-Motor-v1-2, origin xyz=0.03625 -0.00275 -0.1225 rpy=-1.570796326794896 1.6140921240872863e-31 5.290890058994736e-63
- added joint Arm-Forearm-v1_Rigid-8: type fixed, parent Arm-Forearm-v1, child Feetech-Servo-Motor-v1-3, origin xyz=-0.03770996000000019 0.0021637800000000014 0.2657500000000005 rpy=1.5707963267948966 -2.0905669563572298e-64 -2.465190328815666e-32
- added joint Arm-Wrist-v1_Rigid-10: type fixed, parent Arm-Wrist-v1, child Feetech-Servo-Motor-v1-4, origin xyz=-0.038384959999999975 0.0049137800000000394 0.42325000000000124 rpy=1.5707963267948966 -1.0828926805690129e-77 2.101947696487225e-45
- added joint Feetech-Servo-Motor-v1-1_Revolute-5: type revolute, parent Feetech-Servo-Motor-v1-1, child Arm-Bicep-v1, origin xyz=-0.0345 0.03499999999999999 0.0 rpy=1.5707963267948966 -0.0 -2.21816814771825e-32, axis -1.0 -0.0 0.0, limit lower=1.570796 upper=4.712389 effort=1000000 velocity=1000000
- added joint Feetech-Servo-Motor-v1-2_Revolute-7: type revolute, parent Feetech-Servo-Motor-v1-2, child Arm-Forearm-v1, origin xyz=-0.01675000000000003 0.03500000000000004 -7.771561172376097e-18 rpy=1.5707963267948963 -2.4651903288156674e-32 -1.6140921240872852e-31, axis -0.9999999999999989 -1.1102230246251205e-16 -5.338809236774413e-16, limit lower=1.570796 upper=4.712389 effort=1000000 velocity=1000000
- added joint Feetech-Servo-Motor-v1-3_Revolute-9: type revolute, parent Feetech-Servo-Motor-v1-3, child Arm-Wrist-v1, origin xyz=0.03838496 -0.42325 0.0049137799999999995 rpy=-1.5707963267948966 -2.1019476964872216e-45 2.165785361126662e-77, axis -1.0000000000000029 -8.326672684688682e-16 -1.9075514175142588e-16, limit lower=-1.570796 upper=1.570796 effort=1000000 velocity=1000000
- added joint Feetech-Servo-Motor-v1-4_Revolute-11: type revolute, parent Feetech-Servo-Motor-v1-4, child Gripper-Base-Back-v1, origin xyz=0.039384960000000004 -0.49174999999999996 0.00216378 rpy=1.5707963267948966 -0.0 2.465190328815662e-32, axis -2.465190328815662e-32 1.162272669189553e-29 1.0, limit lower=0.0 upper=6.283185 effort=1000000 velocity=1000000
- added joint Feetech-Servo-Motor-v1_Revolute-2: type revolute, parent Feetech-Servo-Motor-v1, child Shoulder-With-Gearbox-V3-v1, origin xyz=5.329070518200751e-17 -0.03499999999999999 0.01675000000000001 rpy=1.5707963267948966 3.1157368034048998e-15 1.559600974533801e-46, axis 4.370308408487244e-32 -1.0 -0.0, limit lower=0.0 upper=3.141593 effort=1000000 velocity=1000000
- added joint Gripper-Base-Back-v1_Rigid-12: type fixed, parent Gripper-Base-Back-v1, child Feetech-Servo-Motor-v1-5, origin xyz=0.0 0.0 0.0020000000000000287 rpy=-1.5707963267948966 1.162272669189553e-29 1.5707963267948966
- added joint Gripper-Base-Back-v1_Rigid-13: type fixed, parent Gripper-Base-Back-v1, child Gripper-Base-Front-Angled-Camera-v1, origin xyz=-0.03 0.029249999999999998 0.03450000000000003 rpy=1.5707963267948966 1.162272669189553e-29 1.5707963267948966
- added joint Gripper-Base-Front-Angled-Camera-v1_Slider-14: type prismatic, parent Gripper-Base-Front-Angled-Camera-v1, child Gripper-Finger-v1, origin xyz=-0.055 0.012000000000000028 -0.01 rpy=1.5707963267948966 -5.36708215504344e-31 5.551115123125783e-17, axis 4.552888492875278e-30 -1.0 -0.0, limit lower=-0.1075 upper=-0.03 effort=1000000 velocity=1000000
- added joint Gripper-Base-Front-Angled-Camera-v1_Slider-15: type prismatic, parent Gripper-Base-Front-Angled-Camera-v1, child Gripper-Finger-v1-1, origin xyz=0.007000000000000002 0.012000000000000028 0.07 rpy=1.5707963267948966 -1.5707963267948966 0, axis 1.0 4.552888492875278e-30 0.0, limit lower=-0.065 upper=0.0 effort=1000000 velocity=1000000
- added joint Shoulder-With-Gearbox-V3-v1_Rigid-4: type fixed, parent Shoulder-With-Gearbox-V3-v1, child Feetech-Servo-Motor-v1-1, origin xyz=0.017425000000000003 0.0 0.03825 rpy=1.5707963267948966 -2.21816814771825e-32 4.370308408487244e-32

Commit message: Huge breakthrough, arm is actually responding to commands

File: lerobot/common/robots/sourccey_v2beta/model/Arm.urdf (robot description, URDF)
Before this commit: robot Arm, 13 links, 12 joints
Links:
- added link Gripper-Gear-ASSEMBLY-TEST-v1, mass 0.06414456756209834; collision mesh filename=meshes/Gripper-Gear-ASSEMBLY-TEST-v1.stl scale=0.001 0.001 0.001; visual mesh filename=meshes/Gripper-Gear-ASSEMBLY-TEST-v1.stl scale=0.001 0.001 0.001
Joints:
- removed joint Feetech-Servo-Motor-v1-1_Revolute-17
- removed joint Feetech-Servo-Motor-v1-2_Revolute-18
- removed joint Feetech-Servo-Motor-v1-3_Revolute-19
- removed joint Feetech-Servo-Motor-v1-4_Revolute-20
- removed joint Feetech-Servo-Motor-v1_Revolute-16
- added joint elbow_flex: type revolute, parent Feetech-Servo-Motor-v1-2, child Arm-Forearm-v1, origin xyz=-0.027296179999999504 0.055126270000000324 0.0349999999999994 rpy=1.5707963267948974 1.1006918418051147e-15 1.5707963267948986, axis 1.0000000000000195 -1.1021770808896294e-15 -1.2116079980132914e-15, limit lower=-1.570796 upper=1.570796 effort=1000000 velocity=1000000
- added joint gripper: type revolute, parent Feetech-Servo-Motor-v1-5, child Gripper-Gear-ASSEMBLY-TEST-v1, origin xyz=0.053451269999998934 -0.03550000000000111 0.012221179999996777 rpy=1.5707963267948966 1.5707963267947707 0, axis 0.0 5.371322496429065e-32 1.0, limit lower=-1.570796 upper=1.570796 effort=1000000 velocity=1000000
- added joint shoulder_lift: type revolute, parent Feetech-Servo-Motor-v1-1, child Arm-Bicep-v1, origin xyz=-0.028296179999999983 0.05962626000000003 0.03499999999999997 rpy=-1.5707963267948968 6.125368411724997e-16 1.570796326794896, axis -1.0000000000000022 -7.984489878059184e-16 -8.556395221968228e-16, limit lower=-1.570796 upper=1.570796 effort=1000000 velocity=1000000
- added joint shoulder_pan: type revolute, parent Feetech-Servo-Motor-v1, child Shoulder-With-Gearbox-V3-v1, origin xyz=0.07705126000000007 0.03499999999999999 -0.010871179999999736 rpy=3.4450928483976567e-16 -3.1900305907108096e-15 9.86076131526302e-32, axis -2.702154975338666e-16 3.4450928483976646e-16 1.0, limit lower=-1.570796 upper=1.570796 effort=1000000 velocity=1000000
- added joint wrist_flex: type revolute, parent Feetech-Servo-Motor-v1-3, child Arm-Wrist-v1, origin xyz=0.02441378 -0.4205 0.07050075 rpy=-3.1415926535897927 -1.5707963267948961 0, axis 0.9999999999999769 -1.3047061815035669e-15 1.2127764798815551e-15, limit lower=-1.570796 upper=1.570796 effort=1000000 velocity=1000000
- added joint wrist_roll: type revolute, parent Feetech-Servo-Motor-v1-4, child Gripper-Base-Back-v1, origin xyz=0.02441378 -0.48625 0.06950075 rpy=1.5707963267949865 -1.5777218104420236e-30 0.0, axis 0.0 8.978648026117131e-14 1.0, limit lower=-3.141593 upper=3.141593 effort=1000000 velocity=1000000
